File: MAXREFDES98_Schematic.brd (EAGLE design)
At the start: 87.8 x 25.4 mm, 34 parts, among them U1 MB110S-TP, U2 MB110S-TP, U3 MAX5969AETB+

Commit message: Added clean version of Nano Pi footprint
Parts:
- U$2: value NANO_PI -> NANO_PI_CLEAN; device Camera_Board_Parts_09_30_2020:NANO_PI -> CameraBoard_Library:NANO_PI_CLEAN
- moved U$2 3.94 mm to (19.7, 0.00)
Changed lines of the file:
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@@
 <element name="L1" library="SD53-3R3-R" package="SD53-3R3-R" value="SD53-3R3-R" x="30.988" y="20.193" smashed="yes" rot="MR270"/>
 <element name="CONN" library="Camera_Board_Parts_09_30_2020" package="TERM_BLOCK_PLUG_8POS_STR_2.5MM" package3d_urn="urn:adsk.eagle:package:24353855/2" value="TERM_BLOCK_PLUG_8POS_STR_2.5MM" x="0.762" y="23.368" smashed="yes" rot="R270"/>
-<element name="U$2" library="Camera_Board_Parts_09_30_2020" package="NANO_PI" package3d_urn="urn:adsk.eagle:package:24353856/1" value="NANO_PI" x="23.622" y="0" smashed="yes"/>
 <element name="R10" library="SparkFun-Resistors" library_urn="urn:adsk.eagle:library:532" package="0603" package3d_urn="urn:adsk.eagle:package:39650/1" value="0" x="4.572" y="18.669" smashed="yes" rot="MR180">
 <attribute name="NAME" x="4.572" y="17.907" size="0.6096" layer="26" font="vector" ratio="20" rot="MR180" align="bottom-center"/>
@@
 <attribute name="VENDOR" value="Bourns Electronics" x="52.578" y="14.605" size="1.778" layer="28" rot="MR180" display="off"/>
 </element>
+<element name="U$2" library="CameraBoard_Library" package="NANO_PI_CLEAN" value="NANO_PI_CLEAN" x="19.685" y="0" smashed="yes"/>
 </elements>
 <signals>
@@
 </signal>
 <signal name="5V_OUT">
-<contactref element="U$2" pad="5V"/>
-<contactref element="U$2" pad="5V_2"/>
 <contactref element="R8" pad="1"/>
 <contactref element="R11" pad="1"/>
@@
 <contactref element="R4" pad="2"/>
 <contactref element="L2_150UH" pad="1"/>
+<contactref element="U$2" pad="5V"/>
+<contactref element="U$2" pad="5V_2"/>
 <wire x1="83.654" y1="1.397" x2="83.704" y2="19.304" width="0" layer="19" extent="1-1"/>
-<wire x1="37.3028" y1="1.27" x2="83.654" y2="1.397" width="0" layer="19" extent="1-1"/>
-<wire x1="34.7628" y1="1.27" x2="37.3028" y2="1.27" width="0" layer="19" extent="1-1"/>
-<wire x1="3.722" y1="13.843" x2="34.7628" y2="1.27" width="0" layer="19" extent="16-16"/>
+<wire x1="44.0944" y1="14.605" x2="83.704" y2="19.304" width="0" layer="19" extent="1-16"/>
+<wire x1="3.722" y1="13.843" x2="44.0944" y2="14.605" width="0" layer="19" extent="16-16"/>
 <wire x1="3.722" y1="21.336" x2="3.722" y2="13.843" width="0" layer="19" extent="16-16"/>
-<wire x1="44.0944" y1="14.605" x2="3.722" y2="13.843" width="0" layer="19" extent="1-16"/>
+<wire x1="30.8258" y1="1.27" x2="3.722" y2="13.843" width="0" layer="19" extent="16-16"/>
+<wire x1="33.3658" y1="1.27" x2="30.8258" y2="1.27" width="0" layer="19" extent="1-1"/>
 </signal>
 <signal name="FB">
@@
 <vertex x="-0.508" y="-0.508"/>
 </polygon>
-<contactref element="U$2" pad="GND"/>
 <contactref element="R10" pad="1"/>
 <contactref element="R9" pad="1"/>
@@
 <contactref element="D3" pad="C"/>
 <contactref element="D4" pad="C"/>
-<wire x1="72.542" y1="5.969" x2="73.5457" y2="20.701" width="0" layer="19" extent="1-1"/>
-<wire x1="72.542" y1="8.509" x2="72.542" y2="5.969" width="0" layer="19" extent="1-1"/>
-<wire x1="83.654" y1="6.477" x2="72.542" y2="5.969" width="0" layer="19" extent="1-1"/>
+<contactref element="U$2" pad="GND"/>
+<wire x1="83.704" y1="21.717" x2="83.654" y2="24.13" width="0" layer="19" extent="1-1"/>
+<wire x1="81.954" y1="14.097" x2="83.704" y2="21.717" width="0" layer="19" extent="1-1"/>
+<wire x1="81.954" y1="11.43" x2="81.954" y2="14.097" width="0" layer="19" extent="1-1"/>
+<wire x1="83.654" y1="6.477" x2="81.954" y2="11.43" width="0" layer="19" extent="1-1"/>
 <wire x1="83.654" y1="3.81" x2="83.654" y2="6.477" width="0" layer="19" extent="1-1"/>
-<wire x1="81.954" y1="11.43" x2="83.654" y2="6.477" width="0" layer="19" extent="1-1"/>
-<wire x1="81.954" y1="14.097" x2="81.954" y2="11.43" width="0" layer="19" extent="1-1"/>
-<wire x1="81.954" y1="1.397" x2="81.954" y2="11.43" width="0" layer="19" extent="1-1"/>
-<wire x1="83.704" y1="21.717" x2="81.954" y2="14.097" width="0" layer="19" extent="1-1"/>
-<wire x1="83.654" y1="24.13" x2="83.704" y2="21.717" width="0" layer="19" extent="1-1"/>
-<wire x1="39.792" y1="18.888" x2="81.954" y2="1.397" width="0" layer="19" extent="1-16"/>
-<wire x1="39.8428" y1="24.13" x2="39.792" y2="18.888" width="0" layer="19" extent="16-16"/>
+<wire x1="81.954" y1="1.397" x2="83.654" y2="3.81" width="0" layer="19" extent="1-1"/>
+<wire x1="72.542" y1="8.509" x2="81.954" y2="11.43" width="0" layer="19" extent="1-1"/>
+<wire x1="72.542" y1="5.969" x2="72.542" y2="8.509" width="0" layer="19" extent="1-1"/>
+<wire x1="73.5457" y1="20.701" x2="83.704" y2="21.717" width="0" layer="19" extent="1-16"/>
+<wire x1="39.792" y1="18.888" x2="73.5457" y2="20.701" width="0" layer="19" extent="16-16"/>
 <wire x1="29.857" y1="13.0555" x2="39.792" y2="18.888" width="0" layer="19" extent="16-16"/>
 <wire x1="29.857" y1="12.5475" x2="29.857" y2="13.0555" width="0" layer="19" extent="16-16"/>
-<wire x1="3.722" y1="16.256" x2="29.857" y2="13.0555" width="0" layer="19" extent="16-16"/>
+<wire x1="35.9058" y1="24.13" x2="29.857" y2="12.5475" width="0" layer="19" extent="16-16"/>
+<wire x1="3.722" y1="16.256" x2="35.9058" y2="24.13" width="0" layer="19" extent="16-16"/>
 <wire x1="3.722" y1="18.669" x2="3.722" y2="16.256" width="0" layer="19" extent="16-16"/>
 </signal>
@@
 <wire x1="22.313" y1="8.509" x2="29.857" y2="11.0235" width="0" layer="19" extent="16-16"/>
 </signal>
-<signal name="3V3">
-<contactref element="U$2" pad="3V3"/>
-</signal>
 <signal name="RD+">
 <contactref element="CONN" pad="5"/>
 <contactref element="U$2" pad="RD+"/>
-<wire x1="7.962" y1="11.268" x2="62.7028" y2="1.27" width="0" layer="19" extent="1-1"/>
+<wire x1="58.7658" y1="1.27" x2="7.962" y2="11.268" width="0" layer="19" extent="1-1"/>
 </signal>
 <signal name="RECT1_IN_MINUS">
@@
 <contactref element="CONN" pad="6"/>
 <contactref element="U$2" pad="RD-"/>
-<wire x1="7.962" y1="8.768" x2="60.1628" y2="1.27" width="0" layer="19" extent="1-1"/>
+<wire x1="56.2258" y1="1.27" x2="7.962" y2="8.768" width="0" layer="19" extent="1-1"/>
 </signal>
 <signal name="TD+">
 <contactref element="CONN" pad="7"/>
 <contactref element="U$2" pad="TD+"/>
-<wire x1="7.962" y1="6.268" x2="67.7828" y2="1.27" width="0" layer="19" extent="1-1"/>
+<wire x1="7.962" y1="6.268" x2="63.8458" y2="1.27" width="0" layer="19" extent="1-1"/>
 </signal>
 <signal name="TD-">
 <contactref element="CONN" pad="8"/>
 <contactref element="U$2" pad="TD-"/>
-<wire x1="7.962" y1="3.768" x2="65.2428" y2="1.27" width="0" layer="19" extent="1-1"/>
+<wire x1="7.962" y1="3.768" x2="61.3058" y2="1.27" width="0" layer="19" extent="1-1"/>
 </signal>
 <signal name="N$6">
@@
 </signal>
 <signal name="LNK">
+<contactref element="R12" pad="2"/>
 <contactref element="U$2" pad="LNK"/>
-<contactref element="R12" pad="2"/>
-<wire x1="65.913" y1="7.024" x2="70.3228" y2="1.27" width="0" layer="19" extent="1-1"/>
+<wire x1="66.3858" y1="1.27" x2="65.913" y2="7.024" width="0" layer="19" extent="1-1"/>
 </signal>
 <signal name="SPD">
+<contactref element="R13" pad="2"/>
 <contactref element="U$2" pad="SPD"/>
-<contactref element="R13" pad="2"/>
-<wire x1="62.992" y1="7.024" x2="72.8628" y2="1.27" width="0" layer="19" extent="1-1"/>
+<wire x1="68.9258" y1="1.27" x2="62.992" y2="7.024" width="0" layer="19" extent="1-1"/>
 </signal>
 <signal name="N$1">
@@
 <wire x1="62.992" y1="8.724" x2="69.698" y2="5.969" width="0" layer="19" extent="1-1"/>
 </signal>
+<signal name="3V3">
+<contactref element="U$2" pad="3V3"/>
+</signal>
 </signals>

Commit message: Update MAXREFDES98_Schematic.brd
Parts:
- moved D2 7.64 mm to (78.9, 22.7)
- moved C2 2.29 mm to (42.7, 10.0)
- moved C3 1.91 mm to (84.7, 1.40)
- moved C4 1.91 mm to (84.7, 3.81)
- moved C5 1.91 mm to (84.7, 6.48)
- moved C6 1.91 mm to (84.7, 11.4)
- moved C7 1.91 mm to (84.7, 14.1)
- moved C8 1.91 mm to (84.7, 24.1)
- moved R4 1.91 mm to (84.7, 19.3)
- moved R5 1.91 mm to (84.7, 16.6)
- moved R6 1.91 mm to (84.7, 21.7)
- moved R7 1.91 mm to (84.7, 8.76)
- moved L2_150UH 1.15 mm to (53.7, 14.5)
- moved U2 0.76 mm to (11.7, 12.4)
- moved R1 0.13 mm to (21.5, 8.64)

Commit message: New Caps
Parts:
- moved C2 3.18 mm to (42.7, 13.2)
- moved D4 0.40 mm to (71.2, 5.59), flipped to the bottom
- moved D3 0.28 mm to (71.2, 8.26), flipped to the bottom
- moved D2 0.13 mm to (78.9, 22.6)
Changed lines of the file:
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@@
 <attribute name="VALUE" x="33.655" y="18.034" size="0.6096" layer="28" font="vector" ratio="20" rot="MR270" align="top-center"/>
 </element>
-<element name="C2" library="EEE-1JA220UP" package="EEE-1JA220UP" value="EEE-1JA220UP" x="42.672" y="10.033" smashed="yes" rot="MR0"/>
+<element name="C2" library="EEE-1JA220UP" package="EEE-1JA220UP" value="EEE-1JA220UP" x="42.672" y="13.208" smashed="yes" rot="MR0"/>
 <element name="D1" library="SMAJ58A-13-F" package="SMAJ58A-13-F" value="SMAJ58A-13-F" x="25.781" y="20.447" smashed="yes" rot="MR270"/>
 <element name="R1" library="SparkFun-Resistors" library_urn="urn:adsk.eagle:library:532" package="0603" package3d_urn="urn:adsk.eagle:package:39650/1" value="619" x="21.463" y="8.636" smashed="yes" rot="MR180">
@@
 <attribute name="VALUE" x="84.709" y="7.874" size="0.6096" layer="27" font="vector" ratio="20" align="top-center"/>
 </element>
-<element name="D2" library="Camera_Board_Parts_09_30_2020" package="SMB_STM-M" value="STPS3L60USMB_STM-M" x="78.867" y="22.733" smashed="yes" rot="MR180">
-<attribute name="BUILT_BY" value="EMA_UL_Team" x="78.867" y="22.733" size="1.778" layer="28" rot="MR180" display="off"/>
-<attribute name="MANUFACTURER_PART_NUMBER" value="STPS3L60U" x="78.867" y="22.733" size="1.778" layer="28" rot="MR180" display="off"/>
-<attribute name="NAME" x="75.5904" y="23.368" size="1.27" layer="26" ratio="6" rot="SMR180"/>
-<attribute name="SOURCELIBRARY" value="StMicro_2011-06-07" x="78.867" y="22.733" size="1.778" layer="28" rot="MR180" display="off"/>
-<attribute name="VALUE" x="77.1398" y="23.368" size="1.27" layer="22" ratio="6" rot="SMR180"/>
-<attribute name="VENDOR" value="STMicroelectronics" x="78.867" y="22.733" size="1.778" layer="28" rot="MR180" display="off"/>
-</element>
-<element name="D3" library="SparkFun-LED" library_urn="urn:adsk.eagle:library:529" package="FKIT-LED-1206" package3d_urn="urn:adsk.eagle:package:39355/1" value="" x="71.12" y="8.509" smashed="yes">
-<attribute name="NAME" x="71.12" y="9.62025" size="0.6096" layer="25" font="vector" ratio="20" align="bottom-center"/>
-<attribute name="VALUE" x="71.12" y="7.39775" size="0.6096" layer="27" font="vector" ratio="20" align="top-center"/>
-</element>
-<element name="D4" library="SparkFun-LED" library_urn="urn:adsk.eagle:library:529" package="FKIT-LED-1206" package3d_urn="urn:adsk.eagle:package:39355/1" value="" x="71.12" y="5.969" smashed="yes">
-<attribute name="NAME" x="71.12" y="7.08025" size="0.6096" layer="25" font="vector" ratio="20" align="bottom-center"/>
-<attribute name="VALUE" x="71.12" y="4.85775" size="0.6096" layer="27" font="vector" ratio="20" align="top-center"/>
+<element name="D2" library="Camera_Board_Parts_09_30_2020" package="SMB_STM-M" value="STPS3L60USMB_STM-M" x="78.867" y="22.606" smashed="yes" rot="MR180">
+<attribute name="BUILT_BY" value="EMA_UL_Team" x="78.867" y="22.606" size="1.778" layer="28" rot="MR180" display="off"/>
+<attribute name="MANUFACTURER_PART_NUMBER" value="STPS3L60U" x="78.867" y="22.606" size="1.778" layer="28" rot="MR180" display="off"/>
+<attribute name="NAME" x="75.5904" y="23.241" size="1.27" layer="26" ratio="6" rot="SMR180"/>
+<attribute name="SOURCELIBRARY" value="StMicro_2011-06-07" x="78.867" y="22.606" size="1.778" layer="28" rot="MR180" display="off"/>
+<attribute name="VALUE" x="77.1398" y="23.241" size="1.27" layer="22" ratio="6" rot="SMR180"/>
+<attribute name="VENDOR" value="STMicroelectronics" x="78.867" y="22.606" size="1.778" layer="28" rot="MR180" display="off"/>
+</element>
+<element name="D3" library="SparkFun-LED" library_urn="urn:adsk.eagle:library:529" package="FKIT-LED-1206" package3d_urn="urn:adsk.eagle:package:39355/1" value="" x="71.247" y="8.255" smashed="yes" rot="MR0">
+<attribute name="NAME" x="71.247" y="9.36625" size="0.6096" layer="26" font="vector" ratio="20" rot="MR0" align="bottom-center"/>
+<attribute name="VALUE" x="71.247" y="7.14375" size="0.6096" layer="28" font="vector" ratio="20" rot="MR0" align="top-center"/>
+</element>
+<element name="D4" library="SparkFun-LED" library_urn="urn:adsk.eagle:library:529" package="FKIT-LED-1206" package3d_urn="urn:adsk.eagle:package:39355/1" value="" x="71.247" y="5.588" smashed="yes" rot="MR0">
+<attribute name="NAME" x="71.247" y="6.69925" size="0.6096" layer="26" font="vector" ratio="20" rot="MR0" align="bottom-center"/>
+<attribute name="VALUE" x="71.247" y="4.47675" size="0.6096" layer="28" font="vector" ratio="20" rot="MR0" align="top-center"/>
 </element>
 <element name="R12" library="SparkFun-Resistors" library_urn="urn:adsk.eagle:library:532" package="0603" package3d_urn="urn:adsk.eagle:package:39650/1" value="470" x="65.913" y="7.874" smashed="yes" rot="R270">
@@
 <wire x1="83.859" y1="3.81" x2="83.859" y2="6.477" width="0" layer="19" extent="1-1"/>
 <wire x1="75.9365" y1="13.589" x2="83.859" y2="6.477" width="0" layer="19" extent="1-1"/>
-<wire x1="38.522" y1="11.383" x2="75.9365" y2="13.589" width="0" layer="19" extent="1-16"/>
-<wire x1="32.766" y1="18.934" x2="38.522" y2="11.383" width="0" layer="19" extent="16-16"/>
+<wire x1="38.522" y1="14.558" x2="75.9365" y2="13.589" width="0" layer="19" extent="1-16"/>
+<wire x1="32.766" y1="18.934" x2="38.522" y2="14.558" width="0" layer="19" extent="16-16"/>
 <wire x1="28.128" y1="20.043" x2="32.766" y2="18.934" width="0" layer="19" extent="16-16"/>
 <wire x1="28.128" y1="14.623" x2="28.128" y2="20.043" width="0" layer="19" extent="16-16"/>
@@
 <wire x1="85.559" y1="3.81" x2="85.559" y2="6.477" width="0" layer="19" extent="1-1"/>
 <wire x1="83.859" y1="1.397" x2="85.559" y2="3.81" width="0" layer="19" extent="1-1"/>
-<wire x1="72.542" y1="8.509" x2="83.859" y2="11.43" width="0" layer="19" extent="1-1"/>
-<wire x1="72.542" y1="5.969" x2="72.542" y2="8.509" width="0" layer="19" extent="1-1"/>
-<wire x1="80.9117" y1="22.733" x2="85.609" y2="21.717" width="0" layer="19" extent="1-16"/>
-<wire x1="38.522" y1="16.983" x2="80.9117" y2="22.733" width="0" layer="19" extent="16-16"/>
-<wire x1="29.857" y1="13.0555" x2="38.522" y2="16.983" width="0" layer="19" extent="16-16"/>
+<wire x1="69.825" y1="8.255" x2="83.859" y2="11.43" width="0" layer="19" extent="1-1"/>
+<wire x1="69.825" y1="5.588" x2="69.825" y2="8.255" width="0" layer="19" extent="1-1"/>
+<wire x1="80.9117" y1="22.606" x2="85.609" y2="21.717" width="0" layer="19" extent="1-16"/>
+<wire x1="38.522" y1="20.158" x2="80.9117" y2="22.606" width="0" layer="19" extent="16-16"/>
+<wire x1="29.857" y1="13.0555" x2="38.522" y2="20.158" width="0" layer="19" extent="16-16"/>
 <wire x1="29.857" y1="12.5475" x2="29.857" y2="13.0555" width="0" layer="19" extent="16-16"/>
 <wire x1="35.9058" y1="24.13" x2="29.857" y2="12.5475" width="0" layer="19" extent="16-16"/>
@@
 <contactref element="D2" pad="1"/>
 <contactref element="L2_150UH" pad="2"/>
-<wire x1="70.651" y1="13.843" x2="76.8223" y2="22.733" width="0" layer="19" extent="1-16"/>
+<wire x1="70.651" y1="13.843" x2="76.8223" y2="22.606" width="0" layer="19" extent="1-16"/>
 <wire x1="66.8115" y1="14.859" x2="70.651" y2="13.843" width="0" layer="19" extent="1-16"/>
 <wire x1="62.2046" y1="14.478" x2="66.8115" y2="14.859" width="0" layer="19" extent="1-1"/>
@@
 <contactref element="R12" pad="1"/>
 <contactref element="D3" pad="A"/>
-<wire x1="65.913" y1="8.724" x2="69.698" y2="8.509" width="0" layer="19" extent="1-1"/>
+<wire x1="65.913" y1="8.724" x2="72.669" y2="8.255" width="0" layer="19" extent="1-1"/>
 </signal>
 <signal name="N$2">
 <contactref element="R13" pad="1"/>
 <contactref element="D4" pad="A"/>
-<wire x1="62.992" y1="8.724" x2="69.698" y2="5.969" width="0" layer="19" extent="1-1"/>
+<wire x1="62.992" y1="8.724" x2="72.669" y2="5.588" width="0" layer="19" extent="1-1"/>
 </signal>
 <signal name="3V3">
