File: MAXREFDES98_Schematic.brd (EAGLE design)
At the start: 72.8 x 25.5 mm, 34 parts, among them U1 MB110S-TP, U2 MB110S-TP, U3 MAX5969AETB+

Commit message: minor changes
Routing:
- net VDD: track 32.7 -> 33.3 mm
- net GND: track 106.0 -> 105.4 mm, vias 6 -> 8
- net PG_EN/SS_INH: track 13.1 -> 13.0 mm, vias 3 -> 1
Changed lines of the file:
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@@
 <wire x1="26.709" y1="7.2135" x2="26.0115" y2="6.516" width="0.3048" layer="16"/>
 <wire x1="26.0115" y1="6.516" x2="24.638" y2="6.516" width="0.3048" layer="16"/>
-<wire x1="20.289" y1="5.969" x2="22.6794" y2="5.969" width="0.3048" layer="1"/>
-<wire x1="22.6794" y1="5.969" x2="23.5684" y2="6.858" width="0.3048" layer="1"/>
+<wire x1="20.289" y1="5.969" x2="22.8064" y2="5.969" width="0.3048" layer="1"/>
+<wire x1="23.5684" y1="6.731" x2="23.5684" y2="6.858" width="0.3048" layer="1"/>
+<wire x1="23.5684" y1="6.731" x2="22.8064" y2="5.969" width="0.3048" layer="1"/>
 <via x="23.5684" y="6.858" extent="1-16" drill="0.35"/>
 <wire x1="23.5684" y1="6.858" x2="24.296" y2="6.858" width="0.3048" layer="16"/>
 <wire x1="24.296" y1="6.858" x2="24.638" y2="6.516" width="0.3048" layer="16"/>
-<wire x1="26.709" y1="7.2135" x2="26.9645" y2="7.2135" width="0.3048" layer="16"/>
-<wire x1="26.9645" y1="7.2135" x2="27.305" y2="6.873" width="0.3048" layer="16"/>
-<via x="27.305" y="6.873" extent="1-16" drill="0.35"/>
-<wire x1="27.305" y1="6.873" x2="27.305" y2="10.541" width="0.3048" layer="1"/>
-<wire x1="27.305" y1="10.541" x2="26.416" y2="11.43" width="0.3048" layer="1"/>
+<wire x1="26.709" y1="7.2135" x2="26.836" y2="7.0865" width="0.3048" layer="16"/>
+<wire x1="26.836" y1="7.0865" x2="26.836" y2="6.834" width="0.3048" layer="16"/>
+<wire x1="27.051" y1="6.492" x2="27.051" y2="6.619" width="0.3048" layer="16"/>
+<wire x1="27.051" y1="6.619" x2="26.836" y2="6.834" width="0.3048" layer="16"/>
+<via x="27.051" y="6.492" extent="1-16" drill="0.35"/>
+<wire x1="27.178" y1="10.668" x2="27.178" y2="6.619" width="0.3048" layer="1"/>
+<wire x1="27.051" y1="6.492" x2="27.178" y2="6.619" width="0.3048" layer="1"/>
+<wire x1="27.178" y1="10.668" x2="26.416" y2="11.43" width="0.3048" layer="1"/>
 <wire x1="27.813" y1="16.14" x2="27.813" y2="17.272" width="0.3048" layer="16"/>
 <wire x1="27.813" y1="17.272" x2="26.613584375" y2="18.471415625" width="0.3048" layer="16"/>
@@
 <contactref element="U3" pad="EP"/>
 <wire x1="26.709" y1="9.2455" x2="25.9335" y2="9.2455" width="0.3048" layer="16"/>
-<wire x1="25.9335" y1="9.2455" x2="25.527" y2="9.652" width="0.3048" layer="16"/>
-<wire x1="25.527" y1="9.652" x2="20.994" y2="9.652" width="0.3048" layer="16"/>
 <wire x1="20.994" y1="9.652" x2="20.994" y2="8.763" width="0.3048" layer="16"/>
 <wire x1="28.3465" y1="8.379" x2="27.48" y2="9.2455" width="0.3048" layer="16"/>
@@
 <wire x1="22.023" y1="12.149" x2="20.605" y2="13.567" width="0.3048" layer="16"/>
 <wire x1="20.605" y1="13.567" x2="19.381" y2="13.567" width="0.3048" layer="16"/>
+<wire x1="23.03" y1="12.149" x2="22.023" y2="12.149" width="0.3048" layer="16"/>
+<wire x1="25.9335" y1="9.2455" x2="23.03" y2="12.149" width="0.3048" layer="16"/>
 </signal>
 <signal name="DET">
@@
 <contactref element="U$1" pad="3"/>
 <contactref element="C8" pad="1"/>
-<wire x1="33.186" y1="7.874" x2="33.0845" y2="7.9755" width="0.3048" layer="16"/>
 <wire x1="37.299" y1="13.081" x2="38.442" y2="11.938" width="0.3048" layer="1"/>
 <wire x1="38.442" y1="11.938" x2="39.5065" y2="11.938" width="0.3048" layer="1"/>
-<wire x1="29.984" y1="8.2295" x2="30.5377" y2="8.2295" width="0.3048" layer="16"/>
-<wire x1="30.5377" y1="8.2295" x2="30.8932" y2="7.874" width="0.3048" layer="16"/>
-<via x="30.8932" y="7.874" extent="1-16" drill="0.35"/>
-<wire x1="30.8932" y1="7.874" x2="32.3314" y2="7.874" width="0.3048" layer="1"/>
-<via x="32.3314" y="7.874" extent="1-16" drill="0.35"/>
-<wire x1="32.3314" y1="7.874" x2="33.186" y2="7.874" width="0.3048" layer="16"/>
 <wire x1="33.186" y1="7.874" x2="33.147" y2="7.913" width="0.3048" layer="16"/>
 <wire x1="33.147" y1="7.913" x2="33.147" y2="8.89" width="0.3048" layer="16"/>
@@
 <wire x1="33.147" y1="8.89" x2="37.299" y2="13.042" width="0.3048" layer="1"/>
 <wire x1="37.299" y1="13.042" x2="37.299" y2="13.081" width="0.3048" layer="1"/>
+<wire x1="29.984" y1="8.2295" x2="30.5055" y2="8.2295" width="0.3048" layer="16"/>
+<wire x1="30.5055" y1="8.2295" x2="30.861" y2="7.874" width="0.3048" layer="16"/>
+<wire x1="30.861" y1="7.874" x2="33.108" y2="7.874" width="0.3048" layer="16"/>
+<wire x1="33.108" y1="7.874" x2="33.147" y2="7.913" width="0.3048" layer="16"/>
 </signal>
 <signal name="5V_OUT">
@@
 <wire x1="32.09" y1="10.633" x2="34.538" y2="13.081" width="0.3048" layer="1"/>
 <wire x1="34.538" y1="13.081" x2="35.599" y2="13.081" width="0.3048" layer="1"/>
-<wire x1="39.839" y1="17.321" x2="39.839" y2="17.526" width="0.3048" layer="1"/>
 <wire x1="53.047" y1="8.382" x2="53.174" y2="8.509" width="0.3048" layer="1"/>
 <wire x1="53.174" y1="8.509" x2="56.515" y2="8.509" width="0.3048" layer="1"/>
@@
 <wire x1="42.418" y1="9.017" x2="41.402" y2="10.033" width="0.3048" layer="16"/>
 <wire x1="4.357" y1="9.906" x2="4.357" y2="7.366" width="0.3048" layer="16"/>
-<wire x1="29.984" y1="8.7375" x2="31.1405" y2="8.7375" width="0.3048" layer="16"/>
-<wire x1="31.1405" y1="8.7375" x2="31.623" y2="8.255" width="0.3048" layer="16"/>
-<wire x1="31.623" y1="8.255" x2="31.623" y2="6.985" width="0.3048" layer="16"/>
-<wire x1="31.623" y1="6.985" x2="29.591" y2="4.953" width="0.3048" layer="16"/>
 <wire x1="24.3488" y1="4.953" x2="20.6658" y2="1.27" width="0.3048" layer="16"/>
-<wire x1="29.591" y1="4.953" x2="24.3488" y2="4.953" width="0.3048" layer="16"/>
+<wire x1="24.3488" y1="4.953" x2="29.591" y2="4.953" width="0.3048" layer="16"/>
 <wire x1="20.6658" y1="1.27" x2="16.6018" y2="5.334" width="0.3048" layer="16"/>
 <wire x1="11.557" y1="6.223" x2="4.826" y2="6.223" width="0.3048" layer="16"/>
@@
 <wire x1="56.769" y1="15.494" x2="54.635" y2="15.494" width="0.3048" layer="1"/>
 <wire x1="54.635" y1="15.494" x2="54.61" y2="15.469" width="0.3048" layer="1"/>
+<wire x1="29.591" y1="4.953" x2="31.242" y2="6.604" width="0.3048" layer="16"/>
+<wire x1="31.242" y1="6.604" x2="31.242" y2="7.112" width="0.3048" layer="16"/>
+<via x="31.242" y="7.112" extent="1-16" drill="0.35"/>
+<wire x1="31.242" y1="7.112" x2="31.242" y2="8.509" width="0.3048" layer="1"/>
+<wire x1="31.242" y1="8.509" x2="30.988" y2="8.763" width="0.3048" layer="1"/>
+<via x="30.988" y="8.763" extent="1-16" drill="0.35"/>
+<wire x1="30.988" y1="8.763" x2="30.9625" y2="8.7375" width="0.3048" layer="16"/>
+<wire x1="30.9625" y1="8.7375" x2="29.984" y2="8.7375" width="0.3048" layer="16"/>
 </signal>
 <signal name="CLS">
@@
 <wire x1="5.676" y1="4.953" x2="8.42800625" y2="4.953" width="0.3048" layer="16"/>
 <wire x1="8.42800625" y1="4.953" x2="8.47" y2="4.911" width="0.3048" layer="16"/>
-<wire x1="8.47" y1="4.911" x2="11.561" y2="4.911" width="0.3048" layer="1"/>
-<wire x1="11.561" y1="4.911" x2="13.654" y2="7.004" width="0.3048" layer="1"/>
+<wire x1="8.47" y1="4.911" x2="11.307" y2="4.911" width="0.3048" layer="1"/>
+<wire x1="13.4" y1="7.004" x2="11.307" y2="4.911" width="0.3048" layer="1"/>
+<wire x1="13.4" y1="7.004" x2="13.654" y2="7.004" width="0.3048" layer="1"/>
 </signal>
 <signal name="RD-">
@@
 <wire x1="30.4" y1="5.033" x2="29.502" y2="5.931" width="0.3048" layer="1"/>
 <wire x1="29.502" y1="5.931" x2="29.502" y2="18.598" width="0.3048" layer="1"/>
-<wire x1="34.886" y1="7.874" x2="34.925" y2="7.835" width="0.3048" layer="16"/>
 <wire x1="32.09" y1="5.033" x2="32.09" y2="5.248" width="0.3048" layer="1"/>
 <wire x1="38.139" y1="17.526" x2="37.123" y2="16.51" width="0.3048" layer="1"/>
@@
 <wire x1="46.692425" y1="7.239" x2="47.581425" y2="8.128" width="0.3048" layer="1"/>
 <wire x1="41.783" y1="6.223" x2="36.537" y2="6.223" width="0.3048" layer="16"/>
-<wire x1="36.537" y1="6.223" x2="34.886" y2="7.874" width="0.3048" layer="16"/>
 <wire x1="32.09" y1="5.248" x2="33.573" y2="6.731" width="0.3048" layer="1"/>
 <wire x1="33.573" y1="6.731" x2="34.925" y2="6.731" width="0.3048" layer="1"/>
@@
 <wire x1="41.783" y1="6.223" x2="42.799" y2="7.239" width="0.3048" layer="1"/>
 <wire x1="42.799" y1="7.239" x2="46.692425" y2="7.239" width="0.3048" layer="1"/>
+<wire x1="36.537" y1="6.223" x2="34.886" y2="7.874" width="0.3048" layer="16"/>
 </signal>
 </signals>
@@
 <mfgpreviewcolor name="substratecolor" color="0xFF786E46"/>
 </mfgpreviewcolors>
+<errors>
+</errors>
 </board>
 </drawing>
