File: camera-shield.sch (EAGLE design)
At the start: 21 parts, among them T1 TG110-S055N2RL

Commit message: Flip ethernet termination, use transformer symbol, clean up repo a little
Parts:
- removed T1: TG110-S055N2RL, CameraBoard_Library:TG110-S055N2RL
- added U$1: ETH-TRANS, ethernet transformer:ETH-TRANS
Connections:
- net ETH_RD_N: now also U$1R.D+; no longer T1.6
- net ETH_RD_P: now also U$1R.D-; no longer T1.8
- net ETH_TD0_GND: now also U$1R.CT; no longer T1.10
- net ETH_TD1_GND: now also U$1T.CT; no longer T1.15
- net ETH_TD_N: now also U$1T.D+; no longer T1.1
- net ETH_TD_P: now also U$1T.D-; no longer T1.3
- net GND: now also U$2.GND_1
- net N$11: now also U$1T.XCT; no longer T1.2
- net N$3: now also U$1R.XCT; no longer T1.7
- net RD_N: now also U$1R.X+; no longer T1.11
- net RD_P: now also U$1R.X-; no longer T1.9
- net TD_N: now also U$1T.X+; no longer T1.16
- net TD_P: now also U$1T.X-; no longer T1.14
Other:
- moved on the sheet: C1, C2, C3, R1, R2
